File: LED_PCB.kicad_sch (KiCad schematic)
At the start: 180 parts, among them J1 +5v Pad, J10 UART Debug, J11 UART Top (RX), J12 UART Bottom (TX), J13 UART Left (RX), J14 UART Right (TX), J15 ENA Pad, J16 MTX Out Conn, J2 +5v Pad, J3 +5v Pad, J4 +5v Pad, J5 GND Pad, J6 GND Pad, J7 GND Pad, J8 GND Pad, J9 ST-Link Conn, P1 USB_C_Plug_USB2.0, Q1 Si2319CDS, Q2 BSS138, SW1 SW_DP3T, SW2 SW_reset, SW3 SW_DPDT_x2, U1 AMS1117-3.3, U2 TPD4EUSB30, U3 STM32F103C8Tx, Y1 8MHz

Commit message: Inited repo
Parts:
- removed P1: USB_C_Plug_USB2.0, Connector_USB:USB_C_Receptacle_Amphenol_12401610E4-2A_CircularHoles, symbol Connector:USB_C_Plug_USB2.0
- added J17: USB_C_Receptacle_USB2.0, LED_PCB_LIB:USB_C_Connector_16P_SMD, symbol Connector:USB_C_Receptacle_USB2.0
- added R12, R13: 5.1k, Resistor_SMD:R_0402_1005Metric, symbol Device:R
- C1, C76: footprint (none) -> Capacitor_Tantalum_SMD:CP_EIA-3216-12_Kemet-S
- C2, C5: footprint Capacitor_SMD:C_0504_1310Metric -> Capacitor_SMD:C_0805_2012Metric
- J9: symbol Connector_Generic:Conn_01x04 -> Connector_Generic:Conn_01x05
- R11: value R -> 1k5; footprint (none) -> Resistor_SMD:R_0402_1005Metric
Connections:
- net +5V: now also J17.A4 (VBUS), J17.A9 (VBUS), J17.B4 (VBUS), J17.B9 (VBUS)
- net GND: now also J17.A1 (GND), J17.A12 (GND), J17.B1 (GND), J17.B12 (GND), J17.S1 (SHIELD), R12.2, R13.2
- net NRST: now also J9.5 (Pin_5); no longer J9.4 (Pin_4)
- net SWCLK: now also J9.3 (Pin_3); no longer J9.2 (Pin_2)
- net SWDIO: now also J9.4 (Pin_4); no longer J9.3 (Pin_3)
- net USB_DM renamed USB_D-
- net USB_D-: now also J17.A7 (D-), J17.B7 (D-)
- net USB_DP renamed USB_D+
- net USB_D+: now also J17.A6 (D+), J17.B6 (D+)
- new net: J17.A5 (CC1), R13.1
- new net: J17.B5 (CC2), R12.1
Other:
- note added: "Как лучше, вывести на програматор 3,3v или 5v грязных?"
- moved on the sheet: C11, J10, J11, J12, J13, J14, J15, R2, R6, R7, R8, SW1A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

Commit message: traced power polygons
Parts:
- removed J16: MTX Out Conn, TestPoint:TestPoint_2Pads_Pitch2.54mm_Drill0.8mm, symbol Connector_Generic:Conn_01x02
- added J16: Matrix_pad, MountingHole:MountingHole_2.2mm_M2_DIN965_Pad_TopOnly, symbol Connector_Generic:Conn_01x01
- added JP1: Jumper_2_Open, Jumper:SolderJumper-2_P1.3mm_Open_TrianglePad1.0x1.5mm, symbol Jumper:Jumper_2_Open
- J11, J12, J13, J14: footprint TestPoint:TestPoint_Loop_D1.80mm_Drill1.0mm_Beaded -> MountingHole:MountingHole_2.2mm_M2_DIN965_Pad_TopOnly
- J15: value ENA Pad -> LED_MATRIX_IN; footprint TestPoint:TestPoint_Loop_D1.80mm_Drill1.0mm_Beaded -> MountingHole:MountingHole_2.2mm_M2_DIN965_Pad_TopOnly
Connections:
- net LED_MATRIX: now also JP1.2 (B)
- net UART2_RX: now also U3.13 (PA3); no longer U3.14 (PA4)
- net UART2_TX: now also U3.12 (PA2); no longer U3.13 (PA3)
- net at J15.1 (Pin_1): now also JP1.1 (A); no longer SW1.2
- net at D67.1 (DOUT): now also J16.1 (Pin_1)

Commit message: traced rawly
Parts:
- added C77: 100n, Capacitor_SMD:C_0201_0603Metric, symbol Device:C
- added J18: ENA_pad, TestPoint:TestPoint_Keystone_5000-5004_Miniature, symbol Connector_Generic:Conn_01x01
- added R14: 10k, Resistor_SMD:R_0402_1005Metric, symbol Device:R
- added SW4: SW_reset, Button_Switch_SMD:SW_Push_1P1T_NO_Vertical_Wuerth_434133025816, symbol Switch:SW_Push
- J9: value ST-Link Conn -> ST-Link Tagcon; symbol Connector_Generic:Conn_01x05 -> Connector_Generic:Conn_01x06
- JP1: value Jumper_2_Open -> EXT_SIGNAL
Connections:
- net +3V3: now also J9.1 (Pin_1), SW1.2, R14.1; no longer SW1.4
- net GND: now also J9.5 (Pin_5), C77.2, SW4.1; no longer J9.1 (Pin_1)
- net LED_MATRIX: no longer JP1.2 (B)
- net NRST: now also J9.3 (Pin_3); no longer J9.5 (Pin_5)
- net SWCLK: now also J9.4 (Pin_4); no longer J9.3 (Pin_3)
- net SWDIO: now also J9.2 (Pin_2); no longer J9.4 (Pin_4)
- net UART2_RX: now also J10.1 (Pin_1); no longer J13.1 (Pin_1)
- net UART2_TX: now also J10.2 (Pin_2); no longer J12.1 (Pin_1)
- net UART3_RX: now also J13.1 (Pin_1); no longer J10.1 (Pin_1)
- net UART3_TX: now also J12.1 (Pin_1); no longer J10.2 (Pin_2)
- net USR_BTN: now reaches U3.28 (PB15)
- net USR_BTN: now also C77.1, R14.2, SW4.2
- net LED_MATRIX_5V: now reaches D4.3 (DIN), Q2.3 (D), R10.1
- net LED_MATRIX_5V: now also JP1.2 (B)
- new net: J18.1 (Pin_1), SW1.4
Other:
- note added: "Level switch"
- note added: "User button"
- note removed: "Как лучше, вывести на програматор 3,3v или 5v грязных?"
- moved on the sheet: R6, R8, SW1A, SW3A
